Commit message: Add Gazebo room navigation stack and tuning
Room worlds/maps, A*+pure pursuit, rviz configs, helper scripts (reset pose, cmd_vel drop check), and diff-drive plugin torque/accel tuning for more reliable turning.

File: src/scout_mini_pro_description/xacro/macro/common_macros.xacro (robot description, xacro)
@@ -43,6 +43,6 @@
     </xacro:macro>
     <!-- ==================== 传感器固定宏 ==================== -->
-    <!-- 参数：传感器名、偏移量、关节名、尺寸、质量、颜色（从主文件传参） -->
-    <xacro:macro name="sensor_fixed" params="sensor_name x y z joint_name size_x size_y size_z mass color_r color_g color_b color_a:=1.0 gazebo_material:=Gazebo/Grey">
+    <!-- 参数：传感器名、偏移量、关节名、尺寸、质量、颜色、可选 rpy（默认 0 0 0，相机需 pitch -90° 使光学轴朝前） -->
+    <xacro:macro name="sensor_fixed" params="sensor_name x y z joint_name size_x size_y size_z mass color_r color_g color_b color_a:=1.0 gazebo_material:=Gazebo/Grey rpy_r:=0 rpy_p:=0 rpy_y:=0">
         <link name="${sensor_name}">
             <!-- 视觉：简化长方体 + 自定义颜色 -->
@@ -69,7 +69,32 @@
             </gazebo>
         </link>
-        <!-- 传感器关节：固定关节（无运动） -->
+        <!-- 传感器关节：固定关节（无运动），rpy 用于相机等需朝向的传感器 -->
         <joint name="${joint_name}" type="fixed">
-            <origin xyz="${x} ${y} ${z}" />
+            <origin xyz="${x} ${y} ${z}" rpy="${rpy_r} ${rpy_p} ${rpy_y}" />
+            <parent link="base_link" />
+            <child link="${sensor_name}" />
+        </joint>
+    </xacro:macro>
+    <!-- 仅 link+joint，不输出 gazebo 块；用于激光等需在同一 link 上合并 material 与 sensor 的情况，避免两个 gazebo 块导致插件不加载 -->
+    <xacro:macro name="sensor_fixed_no_gazebo" params="sensor_name x y z joint_name size_x size_y size_z mass color_r color_g color_b color_a:=1.0 rpy_r:=0 rpy_p:=0 rpy_y:=0">
+        <link name="${sensor_name}">
+            <visual>
+                <origin xyz="0 0 0" />
+                <geometry><box size="${size_x} ${size_y} ${size_z}" /></geometry>
+                <material name="${sensor_name}_color"><color rgba="${color_r} ${color_g} ${color_b} ${color_a}" /></material>
+            </visual>
+            <collision>
+                <origin xyz="0 0 0" />
+                <geometry><box size="${size_x} ${size_y} ${size_z}" /></geometry>
+            </collision>
+            <inertial>
+                <mass value="${mass}" />
+                <inertia ixx="${(1/12)*mass*(size_y**2 + size_z**2)}" ixy="0" ixz="0"
+                         iyy="${(1/12)*mass*(size_x**2 + size_z**2)}" iyz="0"
+                         izz="${(1/12)*mass*(size_x**2 + size_y**2)}" />
+            </inertial>
+        </link>
+        <joint name="${joint_name}" type="fixed">
+            <origin xyz="${x} ${y} ${z}" rpy="${rpy_r} ${rpy_p} ${rpy_y}" />
             <parent link="base_link" />
             <child link="${sensor_name}" />

File: src/scout_mini_pro_description/xacro/macro/gazebo_diff_drive.xacro (robot description, xacro)
@@ -14,6 +14,8 @@
         publish_tf:=true
         publish_wheel_joint_state:=true
-        update_rate:=50.0">
-        <!-- 差速驱动插件：订阅 cmd_vel，发布 odom、TF -->
+        update_rate:=50.0
+        wheel_torque:=300
+        wheel_acceleration:=20.0">
+        <!-- 差速驱动插件：订阅 cmd_vel，发布 odom、TF。扭矩/加速度需足够大才能在仿真中明显转弯（teleop 验证后已调大）。 -->
         <gazebo>
             <plugin name="diff_drive_controller" filename="libgazebo_ros_diff_drive.so">
@@ -30,4 +32,6 @@
                 <publishWheelJointState>${publish_wheel_joint_state}</publishWheelJointState>
                 <updateRate>${update_rate}</updateRate>
+                <wheelTorque>${wheel_torque}</wheelTorque>
+                <wheelAcceleration>${wheel_acceleration}</wheelAcceleration>
             </plugin>
         </gazebo>

File: src/scout_mini_pro_description/xacro/macro/gazebo_sensor_plugin.xacro (robot description, xacro)
@@ -16,5 +16,9 @@
         range_max:=10.0">
         <gazebo reference="${link_ref}">
+            <!-- laser_link 仅保留此一个 gazebo 块，material 与 sensor 同块，避免两块导致 ray_sensor 插件不加载 -->
+            <material>Gazebo/Red</material>
+            <!-- 与教程一致使用 ray，直接发布到全局 /scan，避免“有话题无消息” -->
             <sensor name="laserscan" type="ray">
+                <pose>0 0 0 0 0 0</pose>
                 <always_on>true</always_on>
                 <update_rate>${update_rate}</update_rate>
@@ -28,4 +32,10 @@
                             <max_angle>${angle_max}</max_angle>
                         </horizontal>
+                        <vertical>
+                            <samples>1</samples>
+                            <resolution>1</resolution>
+                            <min_angle>0</min_angle>
+                            <max_angle>0</max_angle>
+                        </vertical>
                     </scan>
                     <range>
@@ -35,11 +45,8 @@
                     </range>
                 </ray>
-                <plugin name="laserscan" filename="libgazebo_ros_ray_sensor.so">
-                    <ros>
-                        <namespace>${robot_namespace}</namespace>
-                        <remapping>~/out:=${topic}</remapping>
-                    </ros>
-                    <output_type>sensor_msgs/LaserScan</output_type>
-                    <frame_name>${frame_name}</frame_name>
+                <!-- Noetic 使用 libgazebo_ros_laser.so（ray_sensor 为 ROS2/新版本，Noetic 中不存在） -->
+                <plugin name="laserscan" filename="libgazebo_ros_laser.so">
+                    <topicName>/scan</topicName>
+                    <frameName>${frame_name}</frameName>
                 </plugin>
             </sensor>
@@ -47,9 +54,10 @@
     </xacro:macro>
     <!-- ==================== 相机插件（Image + CameraInfo） ==================== -->
+    <!-- 使用扁平话题名，避免 camera/camera/... 嵌套：image_raw、camera_info -->
     <xacro:macro name="gazebo_camera_plugin" params="
         robot_namespace:=/scout_mini_pro
         link_ref:=camera_link
-        topic_image:=camera/image_raw
-        topic_info:=camera/camera_info
+        topic_image:=image_raw
+        topic_info:=camera_info
         frame_name:=camera_link
         update_rate:=30.0
@@ -75,4 +83,5 @@
                 </camera>
                 <plugin name="camera_controller" filename="libgazebo_ros_camera.so">
+                    <robotNamespace>${robot_namespace}</robotNamespace>
                     <ros>
                         <namespace>${robot_namespace}</namespace>
@@ -81,6 +90,62 @@
                     </ros>
                     <camera_name>camera</camera_name>
+                    <!-- 插件实际读取 frameName（驼峰），否则 header.frame_id 为空导致 RViz "Frame [] does not exist" -->
+                    <frameName>${frame_name}</frameName>
                     <frame_name>${frame_name}</frame_name>
                     <hack_baseline>0.07</hack_baseline>
+                </plugin>
+            </sensor>
+        </gazebo>
+    </xacro:macro>
+    <!-- ==================== 深度相机插件（Depth Image + PointCloud2，D435 模拟） ==================== -->
+    <xacro:macro name="gazebo_depth_camera_plugin" params="
+        robot_namespace:=/scout_mini_pro
+        link_ref:=camera_link
+        topic_prefix:=camera
+        frame_name:=camera_link
+        update_rate:=30.0
+        width:=640
+        height:=480
+        hfov:=1.0472
+        clip_near:=0.1
+        clip_far:=10.0">
+        <gazebo reference="${link_ref}">
+            <sensor name="depth_camera" type="depth">
+                <always_on>true</always_on>
+                <update_rate>${update_rate}</update_rate>
+                <visualize>true</visualize>
+                <camera name="depth_head">
+                    <horizontal_fov>${hfov}</horizontal_fov>
+                    <image>
+                        <width>${width}</width>
+                        <height>${height}</height>
+                        <format>R8G8B8</format>
+                    </image>
+                    <clip>
+                        <near>${clip_near}</near>
+                        <far>${clip_far}</far>
+                    </clip>
+                </camera>
+                <plugin name="depth_camera_controller" filename="libgazebo_ros_depth_camera.so">
+                    <robotNamespace>${robot_namespace}</robotNamespace>
+                    <ros>
+                        <namespace>${robot_namespace}</namespace>
+                    </ros>
+                    <!-- 父类 GazeboRosCameraUtils 会发布一组 image+camera_info，必须与深度图话题区分，否则 /depth/camera_info 被占导致 RViz No CameraInfo -->
+                    <imageTopicName>rgb/image_raw</imageTopicName>
+                    <cameraInfoTopicName>rgb/camera_info</cameraInfoTopicName>
+                    <alwaysOn>true</alwaysOn>
+                    <updateRate>${update_rate}</updateRate>
+                    <cameraName>${topic_prefix}</cameraName>
+                    <!-- 深度图与 camera_info 独占 depth/image_raw、depth/camera_info，与父类 rgb/ 话题不冲突 -->
+                    <depthImageTopicName>image_raw</depthImageTopicName>
+                    <depthImageCameraInfoTopicName>camera_info</depthImageCameraInfoTopicName>
+                    <pointCloudTopicName>points</pointCloudTopicName>
+                    <!-- 与 RGB 一致：同时提供 frameName/frame_name，确保 header.frame_id 被正确设置 -->
+                    <frameName>${frame_name}</frameName>
+                    <frame_name>${frame_name}</frame_name>
+                    <pointCloudCutoff>${clip_near}</pointCloudCutoff>
+                    <pointCloudCutoffMax>${clip_far}</pointCloudCutoffMax>
+                    <hackBaseline>0.07</hackBaseline>
                 </plugin>
             </sensor>

File: src/scout_mini_pro_description/xacro/main/scout_mini_pro.xacro (robot description, xacro)
@@ -77,6 +77,8 @@
         robot_base_frame="base_footprint"
         publish_tf="true"
-        publish_wheel_joint_state="true"
-        update_rate="50.0" />
+        publish_wheel_joint_state="false"
+        update_rate="50.0"
+        wheel_torque="300"
+        wheel_acceleration="20.0" />
     <xacro:gazebo_joint_state_publisher
         robot_namespace="/scout_mini_pro"
@@ -85,5 +87,10 @@
     <!-- ==================== 7. Gazebo 传感器插件（激光雷达、相机、IMU，由 gazebo_sensor_plugin.xacro 统一管理） ==================== -->
     <xacro:gazebo_laser_plugin robot_namespace="/scout_mini_pro" topic="scan" frame_name="laser_link" />
-    <xacro:gazebo_camera_plugin robot_namespace="/scout_mini_pro" topic_image="camera/image_raw" topic_info="camera/camera_info" frame_name="camera_link" />
-    <xacro:gazebo_imu_plugin robot_namespace="/scout_mini_pro" topic="imu" frame_name="imu_link" />
+    <!-- RGB 相机：可靠发布 image_raw 与 camera_info（libgazebo_ros_camera 较稳定，避免仅依赖深度插件） -->
+    <xacro:gazebo_camera_plugin robot_namespace="/scout_mini_pro" link_ref="camera_link"
+        topic_image="image_raw" topic_info="camera_info" frame_name="camera_link" />
+    <!-- 深度相机：挂在 camera_link，发布深度图、点云（可与 RGB 相机并存） -->
+    <!-- 深度相机话题统一为 /scout_mini_pro/depth/...，避免 /camera/camera/... 嵌套 -->
+    <xacro:gazebo_depth_camera_plugin robot_namespace="/scout_mini_pro" link_ref="camera_link" topic_prefix="depth" frame_name="camera_link" />
+    <!--<xacro:gazebo_imu_plugin robot_namespace="/scout_mini_pro" topic="imu" frame_name="imu_link" />-->
 </robot>

File: src/scout_mini_pro_description/xacro/sensor/camera_d435.xacro (robot description, xacro)
@@ -2,5 +2,5 @@
 <!-- Intel D435深度相机：独立文件，参数可单独修改 -->
 <robot name="camera_d435" xmlns:xacro="http://www.ros.org/wiki/xacro">
-    <!-- 调用通用传感器宏：位置+尺寸+颜色（蓝色） -->
+    <!-- 调用通用传感器宏：位置+尺寸+颜色（蓝色）；恢复到 rpy 全 0 的默认姿态，保持与之前版本一致 -->
     <xacro:sensor_fixed
         sensor_name="camera_link"
@@ -9,4 +9,4 @@
         size_x="0.08" size_y="0.06" size_z="0.04"
         mass="0.1"
-        color_r="0" color_g="0" color_b="1" color_a="0.5" gazebo_material="Gazebo/Blue" />     <!-- D435 约0.1kg -->
+        color_r="0" color_g="0" color_b="1" color_a="0.5" gazebo_material="Gazebo/Blue" />
 </robot>

File: src/scout_mini_pro_description/xacro/sensor/laser_helios.xacro (robot description, xacro)
@@ -1,7 +1,6 @@
 <?xml version="1.0" encoding="UTF-8"?>
-<!-- RS-Helios-16P激光雷达：独立文件 -->
+<!-- RS-Helios-16P激光雷达：独立文件。用 sensor_fixed_no_gazebo 避免 laser_link 出现两个 gazebo 块，material 由 gazebo_laser_plugin 同块输出，确保 ray_sensor 插件能加载 -->
 <robot name="laser_helios" xmlns:xacro="http://www.ros.org/wiki/xacro">
-    <!-- 调用通用传感器宏：位置+尺寸+颜色（红色） -->
-    <xacro:sensor_fixed
+    <xacro:sensor_fixed_no_gazebo
         sensor_name="laser_link"
         x="0" y="0" z="0.22"
@@ -9,4 +8,4 @@
         size_x="0.1" size_y="0.1" size_z="0.05"
         mass="0.8"
-        color_r="1" color_g="0" color_b="0" color_a="0.5" gazebo_material="Gazebo/Red" />     <!-- RS-Helios-16P 约800g -->
+        color_r="1" color_g="0" color_b="0" color_a="0.5" />
 </robot>
