Commit message: Backup full workspace: TD3 offroad, ROS2 migration docs, runs, meshes

File: src/scout_mini_pro_description/xacro/actuator/wheel.xacro (robot description, xacro)
@@ -3,10 +3,12 @@
 <!-- 依赖主文件已定义的全局参数：wheel_diameter, wheel_width, wheel_mass, wheel_x_offset, wheel_y_offset, wheel_z_offset -->
 <robot name="wheel_actuator" xmlns:xacro="http://www.ros.org/wiki/xacro">
-    <!-- 前左轮 -->
+    <!-- 前左轮：被动轮，低摩擦（近似万向轮）；0.15 比 0.1 略稳，仍可灵活转向 -->
     <xacro:wheel wheel_name="front_left_wheel_link" x="${wheel_x_offset}" y="${wheel_y_offset}" z="${wheel_z_offset}"
-                 joint_name="front_left_wheel_joint" wheel_diameter="${wheel_diameter}" wheel_width="${wheel_width}" wheel_mass="${wheel_mass}" />
-    <!-- 前右轮 -->
+                 joint_name="front_left_wheel_joint" wheel_diameter="${wheel_diameter}" wheel_width="${wheel_width}" wheel_mass="${wheel_mass}"
+                 mu1="0.15" mu2="0.15" />
+    <!-- 前右轮：被动轮，低摩擦（近似万向轮） -->
     <xacro:wheel wheel_name="front_right_wheel_link" x="${wheel_x_offset}" y="${-wheel_y_offset}" z="${wheel_z_offset}"
-                 joint_name="front_right_wheel_joint" wheel_diameter="${wheel_diameter}" wheel_width="${wheel_width}" wheel_mass="${wheel_mass}" />
+                 joint_name="front_right_wheel_joint" wheel_diameter="${wheel_diameter}" wheel_width="${wheel_width}" wheel_mass="${wheel_mass}"
+                 mu1="0.15" mu2="0.15" />
     <!-- 后左轮 -->
     <xacro:wheel wheel_name="rear_left_wheel_link" x="${-wheel_x_offset}" y="${wheel_y_offset}" z="${wheel_z_offset}"

File: src/scout_mini_pro_description/xacro/macro/common_macros.xacro (robot description, xacro)
@@ -4,6 +4,6 @@
     <xacro:property name="M_PI" value="3.1415926535897931" />
     <!-- ==================== 车轮通用宏 ==================== -->
-    <!-- 参数：车轮名、偏移量、关节名、车轮尺寸/质量（从主文件传参） -->
-    <xacro:macro name="wheel" params="wheel_name x y z joint_name wheel_diameter wheel_width wheel_mass">
+    <!-- 参数：车轮名、偏移量、关节名、车轮尺寸/质量（从主文件传参）；mu1/mu2 可选，驱动轮用高摩擦、被动轮用低摩擦以免转向时被"抱死" -->
+    <xacro:macro name="wheel" params="wheel_name x y z joint_name wheel_diameter wheel_width wheel_mass mu1:=1.0 mu2:=0.8">
         <link name="${wheel_name}">
             <!-- 视觉：圆柱车轮（旋转90度贴合滚动方向） -->
@@ -27,10 +27,12 @@
                          izz="${0.25*wheel_mass*(wheel_diameter/2)**2 + (1/12)*wheel_mass*wheel_width**2}" />
             </inertial>
-            <!-- Gazebo属性：黑色橡胶材质+高摩擦（简单字符串形式） -->
-            <gazebo reference="${wheel_name}">
-                <material>Gazebo/FlatBlack</material>
-                <mu1>1.0</mu1> <mu2>0.8</mu2>
-            </gazebo>
         </link>
+        <!-- Gazebo属性：黑色橡胶材质，摩擦由调用方指定。
+             注意：<gazebo> 必须是 robot 层级元素，不能嵌在 <link> 内部，
+             否则 URDF->SDF 转换时被静默忽略，mu1/mu2 不生效（转向被前轮抱死的根因） -->
+        <gazebo reference="${wheel_name}">
+            <material>Gazebo/FlatBlack</material>
+            <mu1>${mu1}</mu1> <mu2>${mu2}</mu2>
+        </gazebo>
         <!-- 车轮关节：连续旋转关节 -->
         <joint name="${joint_name}" type="continuous">
